Commit message: Driving done

File: description/robot_core.xacro (robot description, xacro)
@@ -2,14 +2,14 @@
 <robot xmlns:xacro="http://www.ros.org/wiki/xacro" >
     <xacro:include filename="inertial_macros.xacro"/>
-    <material name="white">
+    <material name="White">
         <color rgba="1 1 1 1" />
     </material>
-    <material name="orange">
+    <material name="Orange">
         <color rgba="1 0.3 0.1 1"/>
     </material>
-    <material name="blue">
+    <material name="Blue">
         <color rgba="0.2 0.2 1 1"/>
     </material>
-    <material name="black">
+    <material name="Black">
         <color rgba="0 0 0 1"/>
     </material>
@@ -114,5 +114,5 @@
             </geometry>
         </collision>
-        <xacro:inertial_sphere mass="0.1" radius="0.05">
+        <xacro:inertial_sphere mass="0.2" radius="0.05">
             <origin xyz="0 0 0" rpy="0 0 0"/>
         </xacro:inertial_sphere>
